Commit message: Adding a fourth link with fixed joint in the tip of the robot

File: rc_armsim/urdf/arm4dof.urdf (robot description, URDF)
Before this commit: robot visual, 5 links, 4 joints
Links:
- added link link_round; visual cylinder length=0.03 radius=0.01
- link base_link: geometry visual cylinder length=0.05 radius=0.06
- link link1: geometry visual cylinder length=0.065 radius=0.04
- link link2: geometry visual box size=0.14 0.01 0.02
- link link3: geometry visual box size=0.152 0.01 0.02
- link link4: geometry visual box size=0.032 0.01 0.02
Joints:
- added joint link4_to_link_round: type revolute, parent link4, child link_round, origin xyz=0.032 0.0 -0.03 rpy=0 -0.9 0, axis 0 0 1, limit lower=-1.5 upper=1.5 effort=1000.0 velocity=0.5
- joint base_to_link1: origin xyz=0.0 0.0 0 rpy=0 0 0 -> xyz=0.0 0.0 0.105 rpy=0 0 0
- joint link1_to_link2: limit lower=-1.507 upper=0.22 effort=1000.0 velocity=0.5 -> lower=-1.508 upper=0.22 effort=1000.0 velocity=0.5; origin xyz=0.0 0.0 0.07 rpy=0 0 0 -> xyz=0.0 0.0 0.0 rpy=0 0 0
- joint link2_to_link3: limit lower=-1.5 upper=1.5 effort=1000.0 velocity=0.5 -> lower=-1.508 upper=1.508 effort=1000.0 velocity=0.5; origin xyz=0.2 0.0 0.0 rpy=0 0 0 -> xyz=0.14 0.0 0.0 rpy=0 0 0
- joint link3_to_link4: origin xyz=0.2 0.0 0.0 rpy=0 -0.7 0 -> xyz=0.152 0.0 0.0 rpy=0 0 0; type revolute -> fixed

Commit message: Changing name from link_round to tip

File: rc_armsim/urdf/arm4dof.urdf (robot description, URDF)
Before this commit: robot visual, 6 links, 5 joints
Links:
- removed link link_round
- added link tip; visual cylinder length=0.03 radius=0.01
Joints:
- removed joint link4_to_link_round
- added joint link4_to_tip: type revolute, parent link4, child tip, origin xyz=0.032 0.0 -0.03 rpy=0 -0.9 0, axis 0 0 1, limit lower=-1.5 upper=1.5 effort=1000.0 velocity=0.5

Commit message: Adding a world reference frame

File: rc_armsim/urdf/arm4dof.urdf (robot description, URDF)
Before this commit: robot visual, 6 links, 5 joints
Links:
- added link world
Joints:
- added joint world_to_base: type fixed, parent world, child base_link, origin xyz=0 0 0 rpy=0 0 0, axis 0 0 1
- joint link1_to_link2: limit lower=-1.508 upper=0.22 effort=1000.0 velocity=0.5 -> lower=-1.58 upper=0.22 effort=1000.0 velocity=0.5
- joint link2_to_link3: limit lower=-1.508 upper=1.508 effort=1000.0 velocity=0.5 -> lower=-1.58 upper=1.58 effort=1000.0 velocity=0.5
- joint link3_to_link4: limit lower=-1.5 upper=1.5 effort=1000.0 velocity=0.5 -> (none)
