Commit message: arm4dof simulator is working

File: rc_armsim/urdf/arm.xacro (robot description, xacro)
@@ -37,9 +37,9 @@
     <visual>
       <geometry>
-        <box size="0.032 0.05 0.04"/>
+        <cylinder length="0.04" radius="0.06"/>
       </geometry>
       <origin rpy="0 0 0" xyz="0 -0.0135 0.020"/>
-      <material name="black">
-        <color rgba="0 0 0 1"/>
+      <material name="white">
+        <color rgba="1 1 1 1"/>
       </material>
     </visual>

Commit message: modifying arm.xacro from 4DOF to  3DOF arm, modifying arm_rviz.launch to launch servo2jointstate.py, modifying servo2jointstate.py to be used with the 3DOF arm

File: rc_armsim/urdf/arm.xacro (robot description, xacro)
@@ -10,7 +10,4 @@
 <gazebo_propiedades_link nombre="brazo_link_SI" material="White" />
 <gazebo_propiedades_link nombre="brazo_link_SD" material="White" />
-<gazebo_propiedades_link nombre="antebrazo_link_B" material="White" />
-<gazebo_propiedades_link nombre="antebrazo_link_SI" material="White" />
-<gazebo_propiedades_link nombre="antebrazo_link_SD" material="White" />
 <gazebo_propiedades_link nombre="muneca_link_B" material="White" />
 <gazebo_propiedades_link nombre="muneca_link_SI" material="White" />
@@ -18,13 +15,13 @@
 <gazebo_propiedades_link nombre="muneca_link_P" material="White" />
 <gazebo_propiedades_link nombre="muneca_link_PS" material="White" />
-<gazebo_propiedades_link nombre="pinza_link" material="White" />
-<gazebo_propiedades_link nombre="pinza_link_B" material="White" />
-<gazebo_propiedades_link nombre="pinza_link_SI" material="White" />
-<gazebo_propiedades_link nombre="pinza_link_SD" material="White" />
+<gazebo_propiedades_link nombre="gripper_link" material="White" />
+<gazebo_propiedades_link nombre="gripper_link_B" material="White" />
+<gazebo_propiedades_link nombre="gripper_link_SI" material="White" />
+<gazebo_propiedades_link nombre="gripper_link_SD" material="White" />
 <gazebo_propiedades_joint nombre="base" />
 <gazebo_propiedades_joint nombre="arti1" />
 <gazebo_propiedades_joint nombre="arti2" />
 <gazebo_propiedades_joint nombre="arti3" />
-<gazebo_propiedades_joint nombre="pinza" />
+<gazebo_propiedades_joint nombre="gripper" />
     <macro name="brazo" params="parent *origin">
   <joint name="fixed" type="fixed">
@@ -117,35 +114,4 @@
   <joint name="arti2" type="revolute">
     <parent link="brazo_link"/>
-    <child link="antebrazo_link"/>
-    <origin xyz="0 0 0.104" rpy="0 0 0" />
-    <axis xyz="1 0 0" />
-	<default_limit />
-	<default_dynamics />
-  </joint>
-<!--Antebrazo-->
-<servo nombre="antebrazo" />
-  <joint name="servo_arti2_B" type="fixed">
-    <parent link="antebrazo_link"/>
-    <child link="antebrazo_link_B"/>
-    <origin xyz="0 0 0" rpy="0 0 0" />
-	<axis xyz="1 0 0" />
-  </joint>
-<base nombre="antebrazo" />
-  <joint name="servo_arti2_D" type="fixed">
-    <parent link="antebrazo_link"/>
-    <child link="antebrazo_link_SI"/>
-    <origin xyz="0 0 0" rpy="0 0 0" />
-	<axis xyz="1 0 0" />
-  </joint>
-<soporte nombre="antebrazo" simetrico="1" lado="I" />
-  <joint name="servo_arti2_I" type="fixed">
-    <parent link="antebrazo_link"/>
-    <child link="antebrazo_link_SD"/>
-    <origin xyz="0 0 0" rpy="0 0 0" />
-	<axis xyz="1 0 0" />
-  </joint>
-<soporte nombre="antebrazo" simetrico="-1" lado="D" />
-  <joint name="arti3" type="revolute">
-    <parent link="antebrazo_link"/>
     <child link="muneca_link"/>
     <origin xyz="0 0 0.104" rpy="0 0 0" />
@@ -265,5 +231,5 @@
 	<axis xyz="1 0 0" />
   </joint>
-<!--Pinza fija-->
+<!--gripper fija-->
   <link name="muneca_link_P">
 	<visual>
@@ -316,7 +282,7 @@
     </inertial>
   </link>
-  <joint name="pinza" type="revolute">
-    <parent link="muneca_link"/>
-    <child link="pinza_link"/>
+  <joint name="gripper" type="revolute">
+    <parent link="muneca_link"/>
+    <child link="gripper_link"/>
     <origin xyz="-0.00725 0 0.06" rpy="0 0 0" />
     <axis xyz="0 1 0" />
@@ -324,6 +290,6 @@
 	<default_dynamics />
   </joint>
-<!--Pinza movil-->
-  <link name="pinza_link">
+<!--gripper movil-->
+  <link name="gripper_link">
 	<visual>
       <geometry>
@@ -347,11 +313,11 @@
     </inertial>
   </link>
-  <joint name="servo_pinza_B" type="fixed">
-    <parent link="pinza_link"/>
-    <child link="pinza_link_B"/>
-    <origin xyz="0 0 0" rpy="0 0 0" />
-	<axis xyz="1 0 0" />
-  </joint>
-  <link name="pinza_link_B">
+  <joint name="servo_gripper_B" type="fixed">
+    <parent link="gripper_link"/>
+    <child link="gripper_link_B"/>
+    <origin xyz="0 0 0" rpy="0 0 0" />
+	<axis xyz="1 0 0" />
+  </joint>
+  <link name="gripper_link_B">
 	<visual>
       <geometry>
@@ -375,11 +341,11 @@
     </inertial>
   </link>
-  <joint name="servo_pinza_D" type="fixed">
-    <parent link="pinza_link"/>
-    <child link="pinza_link_SI"/>
-    <origin xyz="0 0 0" rpy="0 0 0" />
-	<axis xyz="1 0 0" />
-  </joint>
-  <link name="pinza_link_SI">
+  <joint name="servo_gripper_D" type="fixed">
+    <parent link="gripper_link"/>
+    <child link="gripper_link_SI"/>
+    <origin xyz="0 0 0" rpy="0 0 0" />
+	<axis xyz="1 0 0" />
+  </joint>
+  <link name="gripper_link_SI">
 	<visual>
       <geometry>
@@ -403,11 +369,11 @@
     </inertial>
   </link>
-  <joint name="servo_pinza_I" type="fixed">
-    <parent link="pinza_link"/>
-    <child link="pinza_link_SD"/>
-    <origin xyz="0 0 0" rpy="0 0 0" />
-	<axis xyz="1 0 0" />
-  </joint>
-  <link name="pinza_link_SD">
+  <joint name="servo_gripper_I" type="fixed">
+    <parent link="gripper_link"/>
+    <child link="gripper_link_SD"/>
+    <origin xyz="0 0 0" rpy="0 0 0" />
+	<axis xyz="1 0 0" />
+  </joint>
+  <link name="gripper_link_SD">
 	<visual>
       <geometry>

File: rc_armsim/urdf/arm_macros.xacro (robot description, xacro)
@@ -43,13 +43,7 @@
     <motorTorqueConstant>1.0</motorTorqueConstant>
  </transmission>
- <transmission type="pr2_mechanism_model/SimpleTransmission" name="arti3_trans">
-    <actuator name="arti3_motor" />
-    <joint name="arti3" />
-    <mechanicalReduction>1.0</mechanicalReduction>
-    <motorTorqueConstant>1.0</motorTorqueConstant>
- </transmission>
- <transmission type="pr2_mechanism_model/SimpleTransmission" name="pinza_trans">
-    <actuator name="pinza_motor" />
-    <joint name="pinza" />
+ <transmission type="pr2_mechanism_model/SimpleTransmission" name="gripper_trans">
+    <actuator name="gripper_motor" />
+    <joint name="gripper" />
     <mechanicalReduction>1.0</mechanicalReduction>
     <motorTorqueConstant>1.0</motorTorqueConstant>
